File: piddle/pcb/piddle.kicad_pcb (KiCad board)
At the start: 2 copper layers, 118 x 104.8 mm, 42 parts, among them J1 Conn_01x03_Socket, J10 Conn_01x03_Socket, J2 Conn_01x03_Socket, J3 Conn_01x03_Socket, J4 Conn_01x03_Socket, J5 Conn_01x03_Socket, J6 Conn_01x03_Socket, J7 Conn_01x03_Socket, J8 Conn_01x03_Socket, J9 Conn_01x03_Socket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

Commit message: Add GPIO silks
Other:
- board text added: "GPIO16"
- board text added: "GPIO17"
- board text added: "GPIO21"
- board text added: "GPIO22"
- board text added: "GPIO25"
- board text added: "GPIO26"
- board text added: "GPIO27"
- board text added: "GPIO32"
- board text added: "GPIO33"
- board text added: "GPIO4"
- board text added: "Phonic Bloom v1 Brandon Skari github.com/ apogaea/piddle"
Changed lines of the file:
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@@
     (property "ki_keywords" "connector")
     (attr through_hole)
-    (fp_text reference "J9" (at 7.802839 3.180137 108) (layer "F.SilkS")
+    (fp_text reference "J9" (at 8.099853 0.647987 108) (layer "F.SilkS")
         (effects (font (size 1 1) (thickness 0.15)))
     )
@@
     (property "ki_keywords" "connector")
     (attr through_hole)
-    (fp_text reference "J10" (at 8.102334 2.342634 144) (layer "F.SilkS")
+    (fp_text reference "J10" (at 8.83869 -0.046462 144) (layer "F.SilkS")
         (effects (font (size 1 1) (thickness 0.15)))
     )
@@
     (property "ki_keywords" "connector")
     (attr through_hole)
-    (fp_text reference "J8" (at 8.145858 2.729671 72) (layer "F.SilkS")
+    (fp_text reference "J8" (at 7.694336 -0.278007 72) (layer "F.SilkS")
         (effects (font (size 1 1) (thickness 0.15)))
     )
@@
     (property "ki_keywords" "connector")
     (attr through_hole)
-    (fp_text reference "J7" (at 8.541858 2.995787 36) (layer "F.SilkS")
+    (fp_text reference "J7" (at 7.805502 0.606691 36) (layer "F.SilkS")
         (effects (font (size 1 1) (thickness 0.15)))
     )
@@
     )
     (stroke (width 0.05) (type solid)) (fill none) (layer "Edge.Cuts"))
+  (gr_text "GPIO33" (at 79.61328 65.096343 36) (layer "F.SilkS")
+    (effects (font (size 1 1) (thickness 0.1)) (justify left bottom))
+  )
+  (gr_text "GPIO22" (at 127.11328 61.596343 -36) (layer "F.SilkS")
+    (effects (font (size 1 1) (thickness 0.1)) (justify left bottom))
+  )
+  (gr_text "GPIO32" (at 109.61328 64.096343) (layer "F.SilkS")
+    (effects (font (size 1 1) (thickness 0.1)) (justify left bottom))
+  )
+  (gr_text "GPIO25" (at 65.61328 86.096343 72) (layer "F.SilkS")
+    (effects (font (size 1 1) (thickness 0.1)) (justify left bottom))
+  )
+  (gr_text "GPIO27" (at 83.61328 141.596343 324) (layer "F.SilkS")
+    (effects (font (size 1 1) (thickness 0.1)) (justify left bottom))
+  )
+  (gr_text "GPIO4" (at 95.61328 157.596343) (layer "F.SilkS")
+    (effects (font (size 1 1) (thickness 0.1)) (justify left bottom))
+  )
+  (gr_text "Phonic Bloom v1\nBrandon Skari\ngithub.com/\napogaea/piddle" (at 58.11328 128.596343 324) (layer "F.SilkS")
+    (effects (font (size 1 1) (thickness 0.1)) (justify left bottom))
+  )
+  (gr_text "GPIO21" (at 142.61328 82.096343 -72) (layer "F.SilkS")
+    (effects (font (size 1 1) (thickness 0.1)) (justify left bottom))
+  )
+  (gr_text "GPIO17" (at 157.11328 113.596343 72) (layer "F.SilkS")
+    (effects (font (size 1 1) (thickness 0.1)) (justify left bottom))
+  )
+  (gr_text "GPIO26" (at 53.11328 111.596343 288) (layer "F.SilkS")
+    (effects (font (size 1 1) (thickness 0.15)))
+  )
+  (gr_text "GPIO16" (at 137.11328 134.596343 36) (layer "F.SilkS")
+    (effects (font (size 1 1) (thickness 0.1)) (justify left bottom))
+  )
   (segment (start 118.899657 95.72272) (end 96.04 95.72272) (width 0.2) (layer "B.Cu") (net 1))
   (segment (start 96.04 95.72272) (end 92.6 92.28272) (width 0.2) (layer "B.Cu") (net 1))
@@
   (segment (start 137.041414 117.68272) (end 118 117.68272) (width 0.2) (layer "F.Cu") (net 33))
   (segment (start 122.987807 138.9) (end 105.189623 138.9) (width 0.2) (layer "B.Cu") (net 34))
-  (segment (start 129.725244 138.013989) (end 123.873818 138.013989) (width 0.2) (layer "B.Cu") (net 34))
   (segment (start 64.11328 101.596343) (end 78.11328 87.596343) (width 0.2) (layer "B.Cu") (net 34))
+  (segment (start 123.873818 136.882619) (end 138.514803 122.241634) (width 0.2) (layer "B.Cu") (net 34))
   (segment (start 137.134356 79.261052) (end 137.134356 98.219179) (width 0.2) (layer "B.Cu") (net 34))
   (segment (start 92.6 138.00272) (end 91.825218 138.00272) (width 0.2) (layer "B.Cu") (net 34))
   (segment (start 78.11328 81.096343) (end 88.11328 71.096343) (width 0.2) (layer "B.Cu") (net 34))
-  (segment (start 144.366229 123.373004) (end 129.725244 138.013989) (width 0.2) (layer "B.Cu") (net 34))
   (segment (start 123.873818 138.013989) (end 122.987807 138.9) (width 0.2) (layer "B.Cu") (net 34))
   (segment (start 105.189623 138.9) (end 97.61328 146.476343) (width 0.2) (layer "B.Cu") (net 34))
   (segment (start 132.089647 74.216343) (end 137.134356 79.261052) (width 0.2) (layer "B.Cu") (net 34))
+  (segment (start 138.514803 122.241634) (end 144.366229 122.241634) (width 0.2) (layer "B.Cu") (net 34))
   (segment (start 78.11328 87.596343) (end 78.11328 81.096343) (width 0.2) (layer "B.Cu") (net 34))
   (segment (start 77.747107 121.73017) (end 64.11328 108.096343) (width 0.2) (layer "B.Cu") (net 34))
@@
   (segment (start 77.747107 123.924609) (end 77.747107 121.73017) (width 0.2) (layer "B.Cu") (net 34))
   (segment (start 91.23328 74.216343) (end 112.61328 74.216343) (width 0.2) (layer "B.Cu") (net 34))
-  (segment (start 144.366229 122.241634) (end 144.366229 123.373004) (width 0.2) (layer "B.Cu") (net 34))
   (segment (start 64.11328 108.096343) (end 64.11328 101.596343) (width 0.2) (layer "B.Cu") (net 34))
   (segment (start 91.825218 138.00272) (end 77.747107 123.924609) (width 0.2) (layer "B.Cu") (net 34))
   (segment (start 137.134356 98.219179) (end 140.866229 101.951052) (width 0.2) (layer "B.Cu") (net 34))
+  (segment (start 123.873818 138.013989) (end 123.873818 136.882619) (width 0.2) (layer "B.Cu") (net 34))
   (segment (start 140.866229 101.951052) (end 140.866229 118.741634) (width 0.2) (layer "B.Cu") (net 34))
   (segment (start 88.11328 71.096343) (end 91.23328 74.216343) (width 0.2) (layer "B.Cu") (net 34))
