File: piddle/pcb/piddle.kicad_sch (KiCad schematic)
At the start: 48 parts, among them J1 Conn_01x03_Socket, J10 Conn_01x03_Socket, J11 Conn_01x02_Socket, J12 Conn_01x02_Socket, J13 Conn_01x02_Pin, J2 Conn_01x03_Socket, J3 Conn_01x03_Socket, J4 Conn_01x03_Socket, J5 Conn_01x03_Socket, J6 Conn_01x03_Socket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

Commit message: Change data line resistor values
Parts:
- R1, R10, R2, R3, R4, R5, R6, R7, R8, R9: value 200 -> 400
Changed lines of the file:
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@@
       (effects (font (size 1.27 1.27)))
     )
-    (property "Value" "200" (at 205.105 140.97 90)
+    (property "Value" "400" (at 205.105 140.97 90)
       (effects (font (size 1.27 1.27)))
     )
@@
       (effects (font (size 1.27 1.27)))
     )
-    (property "Value" "200" (at 76.2 49.53 90)
+    (property "Value" "400" (at 76.2 49.53 90)
       (effects (font (size 1.27 1.27)))
     )
@@
       (effects (font (size 1.27 1.27)))
     )
-    (property "Value" "200" (at 76.2 95.25 90)
+    (property "Value" "400" (at 76.2 95.25 90)
       (effects (font (size 1.27 1.27)))
     )
@@
       (effects (font (size 1.27 1.27)))
     )
-    (property "Value" "200" (at 205.105 48.895 90)
+    (property "Value" "400" (at 205.105 48.895 90)
       (effects (font (size 1.27 1.27)))
     )
@@
       (effects (font (size 1.27 1.27)))
     )
-    (property "Value" "200" (at 205.105 72.39 90)
+    (property "Value" "400" (at 205.105 72.39 90)
       (effects (font (size 1.27 1.27)))
     )
@@
       (effects (font (size 1.27 1.27)))
     )
-    (property "Value" "200" (at 205.105 118.11 90)
+    (property "Value" "400" (at 205.105 118.11 90)
       (effects (font (size 1.27 1.27)))
     )
@@
       (effects (font (size 1.27 1.27)))
     )
-    (property "Value" "200" (at 76.2 141.605 90)
+    (property "Value" "400" (at 76.2 141.605 90)
       (effects (font (size 1.27 1.27)))
     )
@@
       (effects (font (size 1.27 1.27)))
     )
-    (property "Value" "200" (at 205.105 95.25 90)
+    (property "Value" "400" (at 205.105 95.25 90)
       (effects (font (size 1.27 1.27)))
     )
@@
       (effects (font (size 1.27 1.27)))
     )
-    (property "Value" "200" (at 76.2 118.11 90)
+    (property "Value" "400" (at 76.2 118.11 90)
       (effects (font (size 1.27 1.27)))
     )
@@
       (effects (font (size 1.27 1.27)))
     )
-    (property "Value" "200" (at 76.2 72.39 90)
-      (effects (font (size 1.27 1.27)))
-    )
+    (property "Value" "400" (at 76.2 72.39 90)
+      (effects (font (size 1.27 1.27)))
+    )

Commit message: Change LED pins so they work with WLED
Connections:
- net GPIO12: now also R4.1
- net GPIO13: now also R5.1
- net GPIO25: now also R1.1; no longer R3.1
- net GPIO26: now also R2.1; no longer R4.1
- net GPIO27: now also R3.1; no longer R5.1
- net GPIO32: no longer R1.1
- net GPIO33: no longer R2.1
Changed lines of the file:
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@@
     (effects (font (size 1.27 1.27)) (justify left bottom))
   )
-  (label "GPIO32" (at 82.55 47.625 0) (fields_autoplaced)
+  (label "GPIO25" (at 82.55 47.625 0) (fields_autoplaced)
     (effects (font (size 1.27 1.27)) (justify left bottom))
   )
@@
     (effects (font (size 1.27 1.27)) (justify left bottom))
   )
-  (label "GPIO26" (at 82.55 116.205 0) (fields_autoplaced)
+  (label "GPIO12" (at 82.55 116.205 0) (fields_autoplaced)
     (effects (font (size 1.27 1.27)) (justify left bottom))
   )
@@
     (effects (font (size 1.27 1.27)) (justify left bottom))
   )
-  (label "GPIO33" (at 82.55 70.485 0) (fields_autoplaced)
+  (label "GPIO26" (at 82.55 70.485 0) (fields_autoplaced)
     (effects (font (size 1.27 1.27)) (justify left bottom))
   )
@@
     (effects (font (size 1.27 1.27)) (justify right bottom))
   )
-  (label "GPIO25" (at 82.55 93.345 0) (fields_autoplaced)
+  (label "GPIO27" (at 82.55 93.345 0) (fields_autoplaced)
     (effects (font (size 1.27 1.27)) (justify left bottom))
   )
@@
     (effects (font (size 1.27 1.27)) (justify left bottom))
   )
-  (label "GPIO27" (at 81.915 139.7 0) (fields_autoplaced)
+  (label "GPIO13" (at 81.915 139.7 0) (fields_autoplaced)
     (effects (font (size 1.27 1.27)) (justify left bottom))
   )
